File: STM32 with BT Hardware.kicad_sch (KiCad schematic)
At the start: 36 parts, among them J1 Conn_Coaxial, J2 Conn_ARM_SWD_TagConnect_TC2030, J3 USB_C_Receptacle_USB2.0_16P, SW1 SW_Push, U1 STM32WB55CEU6, U2 USBLC6-2SC6, U3 MIC5365-3.3YD5, X1 32.768MHz, X2 32MHz

Commit message: Uploaded some project files
Parts:
- added D1: LED, LED_SMD:LED_0402_1005Metric, symbol Device:LED
- added J2: Conn_01x04, Connector_Molex:Molex_PicoBlade_53048-0410_1x04_P1.25mm_Horizontal, symbol Connector_Generic:Conn_01x04
- added R3, R4, R5: 220R, Resistor_SMD:R_0402_1005Metric, symbol Device:R
- C1: renamed from C18; footprint (none) -> Resistor_SMD:R_0603_1608Metric; Manufacturer (none) -> KYOCERA AVX; Manufacturer part# (none) -> 0603YD475MAT2A
- C10: renamed from C8; footprint (none) -> Resistor_SMD:R_0603_1608Metric; Manufacturer (none) -> KYOCERA AVX; Manufacturer part# (none) -> 0603YD475MAT2A
- C11: renamed from C9; footprint (none) -> Capacitor_SMD:C_0402_1005Metric; Manufacturer (none) -> KYOCERA AVX; Manufacturer part# (none) -> 04023C104KAT2A
- C12: renamed from C10; footprint (none) -> Capacitor_SMD:C_0402_1005Metric; Manufacturer (none) -> KYOCERA AVX; Manufacturer part# (none) -> 04023C104KAT2A
- C13: renamed from C16; footprint (none) -> Capacitor_SMD:C_0402_1005Metric; Manufacturer (none) -> KYOCERA AVX; Manufacturer part# (none) -> 04023C104KAT2A
- C14: renamed from C11; footprint (none) -> Resistor_SMD:R_0603_1608Metric; Manufacturer (none) -> KYOCERA AVX; Manufacturer part# (none) -> 0603YD475MAT2A
- C15: renamed from C14; footprint (none) -> Resistor_SMD:R_0402_1005Metric; Manufacturer (none) -> Murata; Manufacturer part# (none) -> GRM1555C1HR30BA01D
- C16: renamed from C15; footprint (none) -> Resistor_SMD:R_0402_1005Metric; Manufacturer (none) -> Murata; Manufacturer part# (none) -> GRM1555C1HR30WA01D
- C17: renamed from C12; value C -> 10p; footprint (none) -> Resistor_SMD:R_0402_1005Metric; Manufacturer (none) -> KYOCERA AVX; Manufacturer part# (none) -> 04025A100JAT4A
- C18: renamed from C13; value C -> 10p; footprint (none) -> Resistor_SMD:R_0402_1005Metric; Manufacturer (none) -> KYOCERA AVX; Manufacturer part# (none) -> 04025A100JAT4A
- C19: renamed from C17; footprint (none) -> Capacitor_SMD:C_0402_1005Metric; Manufacturer (none) -> KYOCERA AVX; Manufacturer part# (none) -> 04023C104KAT2A
- C2: renamed from C19; footprint (none) -> Resistor_SMD:R_0603_1608Metric; Manufacturer (none) -> KYOCERA AVX; Manufacturer part# (none) -> 0603YD475MAT2A
- C3: renamed from C7; footprint (none) -> Resistor_SMD:R_0603_1608Metric; Manufacturer (none) -> KYOCERA AVX; Manufacturer part# (none) -> 0603YD475MAT2A
- C4: renamed from C1; value 100u -> 100n; footprint (none) -> Capacitor_SMD:C_0402_1005Metric; Manufacturer (none) -> KYOCERA AVX; Manufacturer part# (none) -> 04023C104KAT2A
- C5: renamed from C2; value 100u -> 100n; footprint (none) -> Capacitor_SMD:C_0402_1005Metric; Manufacturer (none) -> KYOCERA AVX; Manufacturer part# (none) -> 04023C104KAT2A
- C6: renamed from C3; value 100u -> 100n; footprint (none) -> Capacitor_SMD:C_0402_1005Metric; Manufacturer (none) -> KYOCERA AVX; Manufacturer part# (none) -> 04023C104KAT2A
- C7: renamed from C4; value 100u -> 100n; footprint (none) -> Capacitor_SMD:C_0402_1005Metric; Manufacturer (none) -> KYOCERA AVX; Manufacturer part# (none) -> 04023C104KAT2A
- C8: renamed from C5; value 100u -> 100n; footprint (none) -> Capacitor_SMD:C_0402_1005Metric; Manufacturer (none) -> KYOCERA AVX; Manufacturer part# (none) -> 04023C104KAT2A
- C9: renamed from C6; value 100u -> 100n; footprint (none) -> Capacitor_SMD:C_0402_1005Metric; Manufacturer (none) -> KYOCERA AVX; Manufacturer part# (none) -> 04023C104KAT2A
- FLT1: Manufacturer (none) -> Wurth; Manufacturer part# (none) -> DLF162500LT-5028A1
- J1: renamed from J3; footprint (none) -> Connector_USB:USB_C_Receptacle_GCT_USB4105-xx-A_16P_TopMnt_Horizontal; Manufacturer (none) -> GCT; Manufacturer part# (none) -> USB4105-GF-A
- J3: renamed from J2; value Conn_ARM_SWD_TagConnect_TC2030 -> TC2030
- J4: renamed from J1; footprint (none) -> Connector_Coaxial:U.FL_Hirose_U.FL-R-SMT-1_Vertical; Manufacturer (none) -> Hirose; Manufacturer part# (none) -> U.FL-R-SMT(01)
- L1: footprint (none) -> Inductor_SMD:L_0402_1005Metric; Manufacturer (none) -> Murata; Manufacturer part# (none) -> LQG15WZ10NJ02D
- L2: footprint (none) -> Inductor_SMD:L_0805_2012Metric; Manufacturer (none) -> Murata; Manufacturer part# (none) -> LQM21FN100M70L
- L3: footprint (none) -> Inductor_SMD:L_0402_1005Metric; Manufacturer (none) -> Murata; Manufacturer part# (none) -> LQG15HS2N7402
- R1: renamed from R3; footprint (none) -> Resistor_SMD:R_0402_1005Metric; Manufacturer (none) -> YAGEO; Manufacturer part# (none) -> RC0603FR-075K1L
- R2: renamed from R4; footprint (none) -> Resistor_SMD:R_0402_1005Metric; Manufacturer (none) -> YAGEO; Manufacturer part# (none) -> RC0603FR-075K1L
- R6: renamed from R1; footprint (none) -> Resistor_SMD:R_0402_1005Metric; Manufacturer (none) -> YAGEO; Manufacturer part# (none) -> RC0603FR-075K1L
- R7: renamed from R2; value 100R -> 220R; footprint (none) -> Resistor_SMD:R_0402_1005Metric; Manufacturer (none) -> YAGEO; Manufacturer part# (none) -> RC0402FR-07221RL
- SW1: footprint (none) -> Button_Switch_SMD:SW_SPST_CK_RS282G05A3; Manufacturer (none) -> C&K; Manufacturer part# (none) -> RS282G05A3SMRT
- U1: renamed from U2; Manufacturer (none) -> STMicroelectronics; Manufacturer part# (none) -> USBLC6-2SC6
- U2: renamed from U3; Manufacturer (none) -> Microchip; Manufacturer part# (none) -> MIC5365-3.3YDS-TR
- U3: renamed from U1; Manufacturer (none) -> STMicroelectronics; Manufacturer part# (none) -> STM32WB55CEU6
- X1: value 32.768MHz -> 32.768kHz; footprint (none) -> Crystal:Crystal_SMD_2012-2Pin_2.0x1.2mm; Disctributor Link (none) -> https://www.mouser.com/ProductDetail/NDK/NX2012SA-32.768K-S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; Manufacturer (none) -> NDK; Manufacturer part# (none) -> NX2012SA-32.768K-STD-MUB-1
- X2: footprint (none) -> Crystal:Crystal_SMD_2016-4Pin_2.0x1.6mm; Manufacturer (none) -> NDK; Manufacturer part# (none) -> NX2016SA-32M-EXS00A-CS06465
Connections:
- net +3V3: now also J2.1 (Pin_1)
- net GND: now also J2.4 (Pin_4), R5.1
- net UART_TX: now reaches U3.11 (PA2)
- net UART_TX: now also R3.2
- net UART_RX: now reaches U3.12 (PA3)
- net UART_RX: now also R4.2
- net LED_A: now reaches U3.16 (PA7)
- net LED_A: now also D1.2 (A)
- removed net USB_CC1: J1.A5 (CC1), J1.A6 (D+), J1.A7 (D-), J1.B6 (D+), J1.B7 (D-), R2.1, U1.1 (I/O1), U1.3 (I/O2), U1.4 (I/O2), U1.6 (I/O1), U3.37 (PA11), U3.38 (PA12)
- net USB_CC2 renamed USBC_CC2
- new net LED_C: D1.1 (K), R5.2
- new net UART_RXC: J2.3 (Pin_3), R4.1
- new net UART_TXC: J2.2 (Pin_2), R3.1
- new net USBC_CC1: J1.A5 (CC1), R2.1
- new net USBC_D+: J1.A6 (D+), J1.B6 (D+), U1.3 (I/O2), U1.4 (I/O2), U3.38 (PA12)
- new net USBC_D-: J1.A7 (D-), J1.B7 (D-), U1.1 (I/O1), U1.6 (I/O1), U3.37 (PA11)
- no-connect marks 2 -> 21
Other:
- note added: "(3.3-1.8)/220=7mA"
- note added: "+5V to 3V3 LDO Regulator"
- note added: "BOOT0 Switch"
- note added: "Henry Munachimso"
- note added: "LSE (32.768kHz) & HSE (32MHz) Crystals"
- note added: "RF Front-End & u.FL Connector"
- note added: "STM32WB BT Hardware Design"
- note added: "STM32WB55 MCU"
- note added: "Tag-Connect SWD-Header"
- note added: "UART Header"
- note added: "USB-C Connector"
- company: (none) -> Henry Munachimso
- title: (none) -> STM32WB BT Hardware Design
- moved on the sheet: C1, C2, U2
